File: menelaos/7-segment-display-v2.sch (KiCad schematic (older format))
At the start: 38 parts, among them J11 Conn_01x02_Male, J12 Conn_01x02_Male, J13 Conn_01x02_Male, J14 Conn_01x02_Male, J15 Conn_01x02_Male, J16 Conn_01x02_Male, J17 Conn_01x02_Male, J18 Conn_01x02_Male, J19 Conn_01x03_Male, J20 Conn_02x07_Counter_Clockwise, J21 Conn_02x07_Counter_Clockwise, U1 74HCT244, U10 HDSP-7503, U12 HDSP-7503, U14 HDSP-7503, U2 74HC4017E, U3 74HC04, U4 74HC4511E, U5 74HCT244, U6 ULN2003, U8 HDSP-7503

Commit message: This is the delivered version. Both the KiCad project and the code are what was delivered to UdK
Parts:
- removed C8: C, Capacitor_THT:C_Disc_D4.3mm_W1.9mm_P5.00mm, symbol Device:C
- removed RV1, RV2, RV3, RV4, RV5, RV6, RV7, RV8: R_POT_TRIM, Potentiometer_THT:Potentiometer_Bourns_3296W_Vertical, symbol Device:R_POT_TRIM
- added C3: C, Capacitor_THT:C_Disc_D4.3mm_W1.9mm_P5.00mm, symbol Device:C
- added H2, H4, H6, H8: MountingHole, MountingHole:MountingHole_3.2mm_M3_Pad_Via, symbol Mechanical:MountingHole
- added J14: Conn_02x07_Counter_Clockwise, knownParts:PinHeader_2x07_P2.54mm_Vertical-counterclockwise, symbol Connector_Generic:Conn_02x07_Counter_Clockwise
- added R24, R25, R26, R27, R36, R37, R38, R39: R, Resistor_THT:R_Axial_DIN0204_L3.6mm_D1.6mm_P7.62mm_Horizontal, symbol Device:R
- added U11, U13, U15, U17: HDSP-7503, Display_7Segment:HDSP-A151, symbol Display_Character:HDSP-7503
- renumbered H2 to H3, H3 to H5, H4 to H7, J19 to J10, J20 to J11, J21 to J13, J11 to J2, J12 to J3, J13 to J4, J14 to J5, J15 to J6, J16 to J7, J17 to J8, J18 to J9, U8 to U10, U10 to U12, U12 to U14, U14 to U16, U1 to U4, U2 to U5, U3 to U6, U4 to U7, U5 to U8, U6 to U9
Connections:
- wire segments 215 -> 264
- no-connect marks 16 -> 18
