File: menelaos/menelaos-v2.sch (KiCad schematic (older format))
At the start: 19 parts, among them J1 Conn_01x05_Male, J10 Conn_01x15_Male, J2 Conn_02x02_Counter_Clockwise, J3 Conn_01x05_Male, J4 Conn_01x05_Male, J5 Conn_01x05_Male, J6 Conn_02x02_Counter_Clockwise, J7 Conn_02x02_Counter_Clockwise, J8 Conn_02x02_Counter_Clockwise, J9 Conn_01x15_Male, U24 ESP32-WROOM-32D

Commit message: This is the delivered version. Both the KiCad project and the code are what was delivered to UdK
Parts:
- removed J10, J9: Conn_01x15_Male, Connector_PinHeader_2.54mm:PinHeader_1x15_P2.54mm_Vertical, symbol Connector:Conn_01x15_Male
- removed J2, J6, J7, J8: Conn_02x02_Counter_Clockwise, knownParts:PinSocket_2x02_P2.54mm_Vertical_CounterClockWise, symbol Connector_Generic:Conn_02x02_Counter_Clockwise
- removed J3, J4, J5: Conn_01x05_Male, Connector_PinHeader_2.54mm:PinHeader_1x05_P2.54mm_Vertical, symbol Connector:Conn_01x05_Male
Connections:
- net hundreds33 is gone; now on net _hundredsBoard: R5.2, R6.1
- net ones33 is gone; now on net _onesBoard: R1.2, R2.1
- net tens33 is gone; now on net _tensBoard: R3.2, R4.1
- net thousands33 is gone; now on net _thousandsBoard: R7.2, R8.1
- no-connect marks 0 -> 10
