File: menelaos/power-v2.sch (KiCad schematic (older format))
At the start: 16 parts, among them Q1 IRF5305-Reverse-Polarity, U16 LM393, U17 OKI-78SR-5v, U18 OKI-78SR-5v

Commit message: This is the delivered version. Both the KiCad project and the code are what was delivered to UdK
Parts:
- removed C9: C, Capacitor_THT:C_Disc_D4.3mm_W1.9mm_P5.00mm, symbol Device:C
- removed RV10, RV9: R_POT_TRIM, Potentiometer_THT:Potentiometer_Bourns_3296W_Vertical, symbol Device:R_POT_TRIM
- removed U17, U18: OKI-78SR-5v, Converter_DCDC:Converter_DCDC_muRata_OKI-78SR_Vertical, symbol ariadne-rescue:OKI-78SR-5v-OpenSourceCelluloid-upuaut-rescue
- added C1: C, Capacitor_THT:C_Disc_D4.3mm_W1.9mm_P5.00mm, symbol Device:C
- added R10, R20, R22, R23: R, Resistor_THT:R_Axial_DIN0204_L3.6mm_D1.6mm_P7.62mm_Horizontal, symbol Device:R
- added U2, U3: L7805, Package_TO_SOT_THT:TO-220-3_Horizontal_TabDown, symbol Regulator_Linear:L7805
- renumbered C1 to C2, R10 to R21, U16 to U1
Connections:
- net +12V: now also R10.1, U2.1 (IN), U3.1 (IN)
- net +5VL: now also C1.1, R22.1, U3.3 (OUT)
- net +5VP: now also U2.3 (OUT)
- net GND: now also C1.2, R20.2, R23.2, U2.2 (GND), U3.2 (GND)
- net at U1.6 (_): now also R10.2, R20.1
- net at U1.5 (+): now also R22.2, R23.1
- net POWER-IN+: no longer names the net of Q1.2 (D), S4.2 (B)
- no-connect marks 4 -> 3
Other:
- note added: "Changed muratas for L7805CV because of availability\n"
